File: experimental/smd_adapters_with_tabs/smd_adapters_with_tabs.kicad_sch (KiCad schematic)
At the start: 9 parts, among them J1 Conn_02x10_Pin, J2 Conn_01x04_Pin, U1 SLG46826G

Commit message: Cleaned up the schematic and layout.
Parts:
- C1, C2: footprint (none) -> Capacitor_SMD:C_0603_1608Metric
- J1: footprint (none) -> greenpack_smd_adapters:PinHeader_2x20
- J2: footprint (none) -> Connector_JST:JST_SH_SM04B-SRSS-TB_1x04-1MP_P1.00mm_Horizontal
- JP1, JP2: footprint (none) -> Jumper:SolderJumper-2_P1.3mm_Open_Pad1.0x1.5mm
- R1, R2: footprint (none) -> Resistor_SMD:R_0603_1608Metric
Other:
- note added: "NOTE: This schematic is provided for documentation only. The actual layout was done manually as a single footprint to simplify panelizing. Importing the schematic into the layout will erase the existing layout."
Changed lines of the file:
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@@
+    (effects (font (size 1.27 1.27)) (justify left bottom))
+  )
+  (text "NOTE: This schematic is provided for documentation only. The actual\nlayout was done manually as a single footprint to simplify panelizing.\nImporting the schematic into the layout will erase the existing layout."
+    (at 51.435 50.8 0)
     (effects (font (size 1.27 1.27)) (justify left bottom))
   )
@@
   )
   (text "This design is compatible with:\n* SLG46827G\n* SLG46826G\n* SLG46827G"
-    (at 80.01 173.355 0)
+    (at 135.89 106.045 0)
     (effects (font (size 1.27 1.27)) (justify left bottom))
   )
@@
       (effects (font (size 1.27 1.27)) (justify left))
     )
-    (property "Footprint" "" (at 76.581 133.604 90)
+    (property "Footprint" "Resistor_SMD:R_0603_1608Metric" (at 76.581 133.604 90)
       (effects (font (size 1.27 1.27)) hide)
     )
@@
       (effects (font (size 1.27 1.27)) hide)
     )
-    (property "Footprint" "" (at 150.495 133.985 0)
+    (property "Footprint" "Jumper:SolderJumper-2_P1.3mm_Open_Pad1.0x1.5mm" (at 150.495 133.985 0)
       (effects (font (size 1.27 1.27)) hide)
     )
@@
       (effects (font (size 1.27 1.27)) hide)
     )
-    (property "Footprint" "" (at 69.85 74.295 0)
+    (property "Footprint" "Jumper:SolderJumper-2_P1.3mm_Open_Pad1.0x1.5mm" (at 69.85 74.295 0)
       (effects (font (size 1.27 1.27)) hide)
     )
@@
       (effects (font (size 1.27 1.27)) hide)
     )
-    (property "Footprint" "" (at 188.595 74.93 0)
+    (property "Footprint" "greenpack_smd_adapters:PinHeader_2x20" (at 188.595 74.93 0)
       (effects (font (size 1.27 1.27)) hide)
     )
@@
       (effects (font (size 1.27 1.27)) (justify left))
     )
-    (property "Footprint" "" (at 60.706 134.239 90)
+    (property "Footprint" "Resistor_SMD:R_0603_1608Metric" (at 60.706 134.239 90)
       (effects (font (size 1.27 1.27)) hide)
     )
@@
       (effects (font (size 1.27 1.27)) (justify left))
     )
-    (property "Footprint" "" (at 117.8052 137.16 0)
+    (property "Footprint" "Capacitor_SMD:C_0603_1608Metric" (at 117.8052 137.16 0)
       (effects (font (size 1.27 1.27)) hide)
     )
@@
       (effects (font (size 1.27 1.27)) (justify left))
     )
-    (property "Footprint" "" (at 101.9302 137.16 0)
+    (property "Footprint" "Capacitor_SMD:C_0603_1608Metric" (at 101.9302 137.16 0)
       (effects (font (size 1.27 1.27)) hide)
     )
@@
       (effects (font (size 1.27 1.27)) hide)
     )
-    (property "Footprint" "" (at 57.15 74.295 0)
-      (effects (font (size 1.27 1.27)) hide)
-    )
+    (property "Footprint" "Connector_JST:JST_SH_SM04B-SRSS-TB_1x04-1MP_P1.00mm_Horizontal" (at 57.15 74.295 0)
+      (effects (font (size 1.27 1.27)) hide)
+    )
