File: experimental/smd_adapters_with_tabs/smd_adapters_with_tabs.kicad_pcb (KiCad board)
At the start: 2 copper layers, 79.8 x 64.6 mm, 34 parts

Commit message: Generated gerbers
Other:
- board text added: "C1,C2: VDD, VDD2 Bypass"
- board text added: "GreenPak TSSOP-20"
- board text added: "R1,R2: I2C pullup"
- board text added: "Recommanded 1mm PCB"
- board text added: "Version 0.3"
- board text removed: "Greenpaks Version 1.02 Use 0.8mm PCB"
Changed lines of the file:
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@@
   (gr_arc (start 161.544 123.444) (mid 162.442026 123.815974) (end 162.814 124.714)
     (stroke (width 0.1) (type default)) (layer "Edge.Cuts"))
-  (gr_text "C1: 0.1u 0603 (VDD bypass)\nC2: 0.1u 0603 (VDD2 bypass)\nR1: SDA pullup to VDD\nR2: SCL pullup to VDD2\nConnector SH 1mm 4P horizontal (QWIIC)\nVDD2: Connects VDD and VDD2\nVCC: Connects QWIIC VCC to VDD." (at 70.104 97.282) (layer "Cmts.User")
+  (gr_text "Version 0.3" (at 149.86 127.508) (layer "F.SilkS")
+    (effects (font (size 1 1) (thickness 0.15)) (justify left))
+  )
+  (gr_text "Recommanded 1mm PCB" (at 163.449 127.508) (layer "F.SilkS")
+    (effects (font (size 1 1) (thickness 0.15)) (justify left))
+  )
+  (gr_text "C1,C2: VDD, VDD2 Bypass" (at 156.845 66.167) (layer "F.SilkS")
+    (effects (font (size 1 1) (thickness 0.15)))
+  )
+  (gr_text "GreenPak TSSOP-20" (at 139.446 127.508) (layer "F.SilkS")
+    (effects (font (size 1 1) (thickness 0.15)))
+  )
+  (gr_text "R1,R2: I2C pullup" (at 135.001 66.04) (layer "F.SilkS")
+    (effects (font (size 1 1) (thickness 0.15)))
+  )
+  (gr_text "C1: 0.1u 0603 (VDD bypass)\nC2: 0.1u 0603 (VDD2 bypass)\nR1: SDA pullup to VDD\nR2: SCL pullup to VDD2\nConnector SH 1mm 4P horizontal (QWIIC)\nVDD2: Connects VDD and VDD2\nVCC: Connects QWIIC VCC to VDD." (at 80.264 99.187) (layer "Cmts.User")
     (effects (font (size 1 1) (thickness 0.15)) (justify left bottom))
   )
-  (gr_text "Greenpaks Version 1.02\nUse 0.8mm PCB" (at 70.104 78.486) (layer "Cmts.User")
-    (effects (font (size 1 1) (thickness 0.15)) (justify left bottom))
-  )

Commit message: Tweaked the layout.
Other:
- board text added: "OSH"

Commit message: Updated gerber.
Parts:
- moved mouse-bite-2.54mm-slot 185.1 mm to (38.9, 23.7)
- moved mouse-bite-2.54mm-slot 185.1 mm to (3.30, -21.2)
- moved REF** 185.1 mm to (30.0, 6.86)
- moved REF** 185.1 mm to (-5.59, -21.1)
- moved REF** 185.1 mm to (-5.59, 6.86)
- moved REF** 185.1 mm to (30.0, -21.1)
- moved REF** 185.1 mm to (12.2, -21.1)
- moved REF** 185.1 mm to (-23.4, -21.1)
- moved REF** 185.1 mm to (-23.4, 6.86)
- moved REF** 185.1 mm to (12.2, 6.86)
- moved mouse-bite-2.54mm-slot 185.1 mm to (30.0, -7.11)
- moved mouse-bite-2.54mm-slot 185.1 mm to (-14.5, -21.1)
- moved mouse-bite-2.54mm-slot 185.1 mm to (38.9, -37.8)
- moved mouse-bite-2.54mm-slot 185.1 mm to (-5.59, 20.8)
- moved mouse-bite-2.54mm-slot 185.1 mm to (-32.3, 23.6)
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